File: hw/rpi.sch (KiCad schematic (older format))
At the start: 11 parts

Commit message: switch to KiCAD 5 (nightly)
Parts:
- removed J?: Write Enable, symbol TEST_2P
- added JP?: Write Enable, symbol Device:Jumper
- DD?: symbol CAT24 -> ic:CAT24
- R? (x5): symbol R -> Device:R
- VT?: symbol DMG2305UX -> ic:DMG2305UX
- VT? (x2): symbol DMMT5401 -> ic:DMMT5401
- XP?: symbol Rpi_40PIN -> rpi_con:Rpi_40PIN
Connections:
- net GND: now also JP?.2
- net at DD?.7 (WP), R?.2: now also JP?.1
Other:
- moved on the sheet: R?, VT?, VT?A, VT?B

Commit message: hw: start stm page
Parts:
- removed JP?: Write Enable, symbol Device:Jumper
Connections:
- net ~HAT_ID_WE: now reaches DD?.7 (WP), R?.2
- net BCM25 renamed CFG_ID2
Other:
- note added: "Use RPi +3.3\nas powe source"
Changed lines of the file:
@@
 	4850 6050 4950 6050
-Wire Wire Line
-	4950 6050 4950 5750
 Wire Wire Line
 	4950 5400 4950 5300
@@
 Text GLabel 6150 3450 2    60   BiDi ~ 0
 BCM12
-Text GLabel 6150 2950 2    60   BiDi ~ 0
-BCM25
+Text GLabel 6150 2950 2    60   Input ~ 0
+CFG_ID2
 Wire Wire Line
 	6150 2950 5250 2950
@@
 Wire Wire Line
 	4200 8700 4500 8700
-$Comp
-L Device:Jumper JP?
-U 1 1 5AC1291D
-P 5250 6150
-F 0 "JP?" V 5204 6276 50  0000 L CNN
-F 1 "Write Enable" V 5295 6276 50  0000 L CNN
-F 2 "" H 5250 6150 50  0001 C CNN
-F 3 "~" H 5250 6150 50  0001 C CNN
-	1    5250 6150
-	0    1    1    0
-$EndComp
-Wire Wire Line
-	5100 6550 5250 6550
-Wire Wire Line
-	5250 6550 5250 6450
-Connection ~ 5100 6550
-Wire Wire Line
-	5250 5850 5250 5750
-Wire Wire Line
-	5250 5750 4950 5750
-Connection ~ 4950 5750
-Wire Wire Line
-	4950 5750 4950 5700
+Wire Wire Line
+	4950 5700 4950 6050
+Text GLabel 5400 6050 2    60   Input ~ 0
+~HAT_ID_WE
+Wire Wire Line
+	5400 6050 4950 6050
+Connection ~ 4950 6050
+$Comp
+L power:+3.3V #PWR?
+U 1 1 5AC14350
+P 5650 8000
+F 0 "#PWR?" H 5650 7850 50  0001 C CNN
+F 1 "+3.3V" H 5665 8173 50  0000 C CNN
+F 2 "" H 5650 8000 50  0001 C CNN
+F 3 "" H 5650 8000 50  0001 C CNN
+	1    5650 8000
+	1    0    0    -1
+$EndComp
+$Comp
+L power:+3.3VP #PWR?
+U 1 1 5AC148A8
+P 5950 8000
+F 0 "#PWR?" H 6100 7950 50  0001 C CNN
+F 1 "+3.3VP" H 5950 8100 50  0000 C CNN
+F 2 "" H 5950 8000 50  0001 C CNN
+F 3 "" H 5950 8000 50  0001 C CNN
+	1    5950 8000
+	1    0    0    -1
+$EndComp
+Wire Wire Line
+	5650 8000 5650 8100
+Wire Wire Line
+	5650 8100 5950 8100
+Wire Wire Line
+	5950 8100 5950 8000
+$Comp
+L power:PWR_FLAG #FLG?
+U 1 1 5AC179FB
+P 6250 8000
+F 0 "#FLG?" H 6250 8075 50  0001 C CNN
+F 1 "PWR_FLAG" H 6250 8174 50  0000 C CNN
+F 2 "" H 6250 8000 50  0001 C CNN
+F 3 "" H 6250 8000 50  0001 C CNN
+	1    6250 8000
+	1    0    0    -1
+$EndComp
+Wire Wire Line
+	5950 8100 6250 8100
+Wire Wire Line
+	6250 8100 6250 8000
+Connection ~ 5950 8100
+Text Notes 5650 8350 0    60   ~ 0
+Use RPi +3.3\nas powe source
 $EndSCHEMATC

Commit message: hw: update libs
Parts:
- removed VT?: DMMT5401, symbol ic:DMMT5401
- removed VT?: DMMT5401, TO_SOT_Packages_SMD:SOT-23-6_Handsoldering, symbol ic:DMMT5401
- added VT? (x2): DMMT5401, Package_TO_SOT_SMD:SOT-23-6_Handsoldering, symbol hat-ic:DMMT5401
- DD?: symbol ic:CAT24 -> hat-ic:CAT24
- VT?: symbol ic:DMG2305UX -> hat-ic:DMG2305UX
- XP?: symbol rpi_con:Rpi_40PIN -> rpi-conn:Rpi_40PIN
Connections:
- net +5V: now also VT?.6 (E1)
- net +5VP: now also VT?.5 (E2)
- net at R?.1, VT?.1 (G): now also VT?.4 (C2)
- net at R?.1: now also VT?.1 (C1), VT?.2 (B1), VT?.3 (B2)
Changed lines of the file:
@@
 $EndDescr
 $Comp
-L rpi_con:Rpi_40PIN XP?
+L rpi-conn:Rpi_40PIN XP?
 U 1 1 5AAFFE0B
 P 4400 2900
@@
 	2800 3050 3550 3050
 $Comp
-L ic:CAT24 DD?
+L hat-ic:CAT24 DD?
 U 1 1 5AB0087D
 P 4300 6300
@@
 	3550 2650 2800 2650
 $Comp
-L ic:DMG2305UX VT?
+L hat-ic:DMG2305UX VT?
 U 1 1 5AB12B0E
 P 4300 8350
@@
 Wire Wire Line
 	4800 9450 4800 9550
-$Comp
-L ic:DMMT5401 VT?
-U 1 1 5AB144D9
-P 3900 8700
-F 0 "VT?" H 4100 8750 50  0000 L CNN
-F 1 "DMMT5401" H 4100 8650 50  0000 L CNN
-F 2 "" H 4100 8800 50  0001 C CNN
-F 3 "" H 3900 8700 50  0001 C CNN
-	1    3900 8700
-	-1   0    0    1
-$EndComp
-$Comp
-L ic:DMMT5401 VT?
-U 2 1 5AB14574
-P 4700 8700
-F 0 "VT?" H 4900 8750 50  0000 L CNN
-F 1 "DMMT5401" H 4900 8650 50  0000 L CNN
-F 2 "TO_SOT_Packages_SMD:SOT-23-6_Handsoldering" H 4900 8800 50  0001 C CNN
-F 3 "" H 4700 8700 50  0001 C CNN
-	2    4700 8700
-	1    0    0    1
-$EndComp
 $Comp
 L power:+5VP #PWR011
@@
 Text Notes 5650 8350 0    60   ~ 0
 Use RPi +3.3\nas powe source
+$Comp
+L hat-ic:DMMT5401 VT?
+U 1 1 5AC552B8
+P 3900 8700
+F 0 "VT?" H 4090 8654 50  0000 L CNN
+F 1 "DMMT5401" H 4090 8745 50  0000 L CNN
+F 2 "Package_TO_SOT_SMD:SOT-23-6_Handsoldering" H 4100 8800 50  0001 C CNN
+F 3 "" H 3900 8700 50  0001 C CNN
+	1    3900 8700
+	-1   0    0    1
+$EndComp
+$Comp
+L hat-ic:DMMT5401 VT?
+U 2 1 5AC553C3
+P 4700 8700
+F 0 "VT?" H 4891 8654 50  0000 L CNN
+F 1 "DMMT5401" H 4891 8745 50  0000 L CNN
+F 2 "Package_TO_SOT_SMD:SOT-23-6_Handsoldering" H 4900 8800 50  0001 C CNN
+F 3 "" H 4700 8700 50  0001 C CNN
+	2    4700 8700
+	1    0    0    1
+$EndComp
 $EndSCHEMATC

Commit message: hw: sch ready
Parts:
- gave numbers to parts that had none: 9
Changed lines of the file:
@@
 $EndDescr
 $Comp
-L rpi-conn:Rpi_40PIN XP?
+L rpi-conn:Rpi_40PIN XP1
 U 1 1 5AAFFE0B
 P 4400 2900
-F 0 "XP?" H 3850 4100 60  0000 C CNN
+F 0 "XP1" H 3850 4100 60  0000 C CNN
 F 1 "Rpi_40PIN" H 4450 1700 60  0000 C CNN
 F 2 "" H 4050 3000 60  0001 C CNN
@@
 	2800 3050 3550 3050
 $Comp
-L hat-ic:CAT24 DD?
+L hat-ic:CAT24 DD1
 U 1 1 5AB0087D
 P 4300 6300
-F 0 "DD?" H 4050 6750 60  0000 C CNN
+F 0 "DD1" H 4050 6750 60  0000 C CNN
 F 1 "CAT24C32" H 4300 5850 60  0000 C CNN
 F 2 "" V 2700 7750 60  0001 C CNN
@@
 	5100 5200 5100 5300
 $Comp
-L Device:R R?
+L Device:R R1
 U 1 1 5AB0176B
 P 4950 5550
-F 0 "R?" V 5030 5550 50  0000 C CNN
+F 0 "R1" V 5030 5550 50  0000 C CNN
 F 1 "1k" V 4950 5550 50  0000 C CNN
 F 2 "" V 4880 5550 50  0001 C CNN
@@
 	2850 6150 3300 6150
 $Comp
-L Device:R R?
+L Device:R R2
 U 1 1 5AB01D57
 P 3200 5800
-F 0 "R?" V 3400 5800 50  0000 C CNN
+F 0 "R2" V 3400 5800 50  0000 C CNN
 F 1 "3.9k" V 3200 5800 50  0000 C CNN
 F 2 "" V 3130 5800 50  0001 C CNN
@@
 $EndComp
 $Comp
-L Device:R R?
+L Device:R R3
 U 1 1 5AB01DDA
 P 3300 5800
-F 0 "R?" V 3500 5800 50  0000 C CNN
+F 0 "R3" V 3500 5800 50  0000 C CNN
 F 1 "3.9k" V 3300 5800 50  0000 C CNN
 F 2 "" V 3230 5800 50  0001 C CNN
@@
 	3550 2650 2800 2650
 $Comp
-L hat-ic:DMG2305UX VT?
+L hat-ic:DMG2305UX VT1
 U 1 1 5AB12B0E
 P 4300 8350
-F 0 "VT?" V 4550 8450 50  0000 L CNN
+F 0 "VT1" V 4550 8450 50  0000 L CNN
 F 1 "DMG2305UX" V 4550 7950 50  0000 L CNN
 F 2 "TO_SOT_Packages_SMD:SOT-23_Handsoldering" H 4500 8450 50  0001 C CNN
@@
 $EndComp
 $Comp
-L Device:R R?
+L Device:R R5
 U 1 1 5AB13830
 P 4800 9300
-F 0 "R?" V 4880 9300 50  0000 C CNN
+F 0 "R5" V 4880 9300 50  0000 C CNN
 F 1 "47k" V 4800 9300 50  0000 C CNN
 F 2 "" V 4730 9300 50  0001 C CNN
@@
 $EndComp
 $Comp
-L Device:R R?
+L Device:R R4
 U 1 1 5AB13B9E
 P 3800 9300
-F 0 "R?" V 3880 9300 50  0000 C CNN
+F 0 "R4" V 3880 9300 50  0000 C CNN
 F 1 "10k" V 3800 9300 50  0000 C CNN
 F 2 "" V 3730 9300 50  0001 C CNN
@@
 Connection ~ 4950 6050
 $Comp
-L power:+3.3V #PWR?
+L power:+3.3V #PWR013
 U 1 1 5AC14350
 P 5650 8000
-F 0 "#PWR?" H 5650 7850 50  0001 C CNN
+F 0 "#PWR013" H 5650 7850 50  0001 C CNN
 F 1 "+3.3V" H 5665 8173 50  0000 C CNN
 F 2 "" H 5650 8000 50  0001 C CNN
@@
 $EndComp
 $Comp
-L power:+3.3VP #PWR?
+L power:+3.3VP #PWR015
 U 1 1 5AC148A8
 P 5950 8000
-F 0 "#PWR?" H 6100 7950 50  0001 C CNN
+F 0 "#PWR015" H 6100 7950 50  0001 C CNN
 F 1 "+3.3VP" H 5950 8100 50  0000 C CNN
 F 2 "" H 5950 8000 50  0001 C CNN
@@
 	5950 8100 5950 8000
 $Comp
-L power:PWR_FLAG #FLG?
+L power:PWR_FLAG #FLG01
 U 1 1 5AC179FB
 P 6250 8000
-F 0 "#FLG?" H 6250 8075 50  0001 C CNN
+F 0 "#FLG01" H 6250 8075 50  0001 C CNN
 F 1 "PWR_FLAG" H 6250 8174 50  0000 C CNN
 F 2 "" H 6250 8000 50  0001 C CNN
@@
 Use RPi +3.3\nas powe source
 $Comp
-L hat-ic:DMMT5401 VT?
+L hat-ic:DMMT5401 VT2
 U 1 1 5AC552B8
 P 3900 8700
-F 0 "VT?" H 4090 8654 50  0000 L CNN
+F 0 "VT2" H 4090 8654 50  0000 L CNN
 F 1 "DMMT5401" H 4090 8745 50  0000 L CNN
 F 2 "Package_TO_SOT_SMD:SOT-23-6_Handsoldering" H 4100 8800 50  0001 C CNN
@@
 $EndComp
 $Comp
-L hat-ic:DMMT5401 VT?
+L hat-ic:DMMT5401 VT2
 U 2 1 5AC553C3
 P 4700 8700
-F 0 "VT?" H 4891 8654 50  0000 L CNN
+F 0 "VT2" H 4891 8654 50  0000 L CNN
 F 1 "DMMT5401" H 4891 8745 50  0000 L CNN
 F 2 "Package_TO_SOT_SMD:SOT-23-6_Handsoldering" H 4900 8800 50  0001 C CNN
